File: Hardware/KiCad/PC6 Connector/PC6 Connector.kicad_pcb (KiCad board)
At the start: 2 copper layers, 35 x 17.5 mm, 8 parts, among them J1 PC-6 Connector, J2 PCUI Port

Commit message: Updates to PCBs, added 3D models for molds for 702P and 700/770; Update to PC-6 PCB and PB-700 mold; Assembly instruction updates, model updates (track .step/.stl via Git LFS)
Other:
- board text added: "N1UGK REV 1.6"
- board text removed: "N1UGK REV 1.5"
Changed lines of the file:
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@@
 	)
 	(gr_rect
-		(start 121.25 90.5)
-		(end 123.75 91.5)
+		(start 121.6 98)
+		(end 124.1 99)
 		(stroke
 			(width 0.1)
@@
 		)
 	)
-	(gr_text "N1UGK REV 1.5"
+	(gr_text "N1UGK REV 1.6"
 		(at 118.65 104.55 0)
 		(layer "B.SilkS")
